File: w5500.kicad_sch (KiCad schematic)
At the start: 21 parts, among them J6 HR911105A, U5 W5500, Y1 X201625MOB4SI - 25Mhz

Commit message: update
Parts:
- C21: value 4.7µF - CL05A475MP5NRNC -> 4.7µF
- Y1: value X201625MOB4SI - 25Mhz -> X201625MOB4SI 25Mhz
Changed lines of the file:
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@@
 			)
 		)
-		(property "Value" "4.7µF - CL05A475MP5NRNC"
+		(property "Value" "4.7µF"
 			(at 248.92 130.8099 0)
 			(effects
@@
 			)
 		)
-		(property "Value" "X201625MOB4SI - 25Mhz"
+		(property "Value" "X201625MOB4SI  25Mhz"
 			(at 203.962 29.21 90)
 			(effects
