File: kicad/ESPrelay.kicad_sch (KiCad schematic)
At the start: 38 parts, among them J1 POWER_INPUT, J2 GT-USB-7051A, J3 MOLEX 545480671, J4 RJ12, J5 A7670C MODULE, Q1 TBD62083AFG_EL, SW1 SW_Push, U1 MC7805BD2TR4G, U2 ESP32-S3-WROOM-1-N4, U3 LF33CDT-TR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

Commit message: minor bug update. add daughter pcb initial commit
Parts:
- added J14: TS02115B0000G, symbol Connector:Screw_Terminal_01x02
- J1: value POWER_INPUT -> MCV_1,5_2-G-3.5
Changed lines of the file:
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@@
 			)
 		)
-		(property "Value" "POWER_INPUT"
-			(at 19.812 172.466 0)
+		(property "Value" "MCV_1,5_2-G-3.5"
+			(at 25.146 178.054 0)
 			(effects
 				(font
@@
 		(on_board yes)
 		(dnp no)
-		(fields_autoplaced yes)
 		(property "Reference" "#FLG01"
 			(at 34.29 169.545 0)
@@
 		)
 		(property "Value" "PWR_FLAG"
-			(at 34.29 166.37 0)
+			(at 21.844 171.958 0)
 			(effects
 				(font
@@
 					(unit 1)
 				)
+			)
+		)
+	)
+	(symbol
+		(lib_id "Connector:Screw_Terminal_01x02")
+		(at 22.86 163.83 180)
+		(unit 1)
+		(exclude_from_sim yes)
+		(in_bom no)
+		(on_board no)
+		(dnp no)
+		(fields_autoplaced yes)
+		(property "Reference" "J14"
+			(at 22.86 154.94 0)
+			(effects
+				(font
+					(size 1.27 1.27)
+				)
+			)
+		)
+		(property "Value" "TS02115B0000G"
+			(at 22.86 157.48 0)
+			(effects
+				(font
+					(size 1.27 1.27)
+				)
+			)
+		)
+		(property "Footprint" ""
+			(at 22.86 163.83 0)
+			(effects
+				(font
+					(size 1.27 1.27)
+				)
+				(hide yes)
+			)
+		)
+		(property "Datasheet" "~"
+			(at 22.86 163.83 0)
+			(effects
+				(font
+					(size 1.27 1.27)
+				)
+				(hide yes)
+			)
+		)
+		(property "Description" "Generic screw terminal, single row, 01x02, script generated (kicad-library-utils/schlib/autogen/connector/)"
+			(at 22.86 163.83 0)
+			(effects
+				(font
+					(size 1.27 1.27)
+				)
+				(hide yes)
+			)
+		)
+		(pin "1"
+		)
+		(pin "2"
+		)
+		(instances
+			(project ""
+				(path "/69ed8f4f-6a33-4210-b2ac-8a5f3a02835d"
+					(reference "J14")
+					(unit 1)
+				)
