File: kicad/daughter_4relays/input.kicad_sch (KiCad schematic)
At the start: 12 parts, among them J11 MCV_1,5_6-G-3.5, J12 TS06115B0000GAMPHENOL, U6 TCMT4100

Commit message: minor bug update. add daughter pcb initial commit
Parts:
- removed J12: TS06115B0000GAMPHENOL, symbol Connector:Screw_Terminal_01x06
- J4: renamed from J11; value MCV_1,5_6-G-3.5 -> Screw_Terminal_01x06
- renumbered JP1 to JP3, R24 to R10, R17 to R3, R18 to R4, R19 to R5, R20 to R6, R21 to R7, R22 to R8, R23 to R9, U6 to U2
Other:
- note removed: "TS06115B0000GAMPHENOL ANYTEK"
- note removed: "mating connector :"
- moved on the sheet: J4, JP3, R10, R3, R4, R5, R6, R7, R8, R9, U2A, U2B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
